File: SolarCar26_Red_Lights_PCB.kicad_sch (KiCad schematic)
At the start: 8 parts, among them J1 Conn_01x02

Commit message: Add files via upload
Connections:
- net +12V: now reaches J1.1 (Pin_1)
- net +12V: now also D1.2 (A); no longer R1.1
- net at R1.2: now also D6.1 (K); no longer D1.2 (A)
- net GND: now reaches J1.2 (Pin_2)
- net GND: now also R1.1; no longer D6.1 (K)
Other:
- moved on the sheet: R1
Changed lines of the file:
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@@
-	(wire
-		(pts
-			(xy 97.79 44.45) (xy 97.79 57.15)
-		)
-		(stroke
-			(width 0)
-			(type default)
-		)
-	)
-	(wire
-		(pts
-			(xy 97.79 64.77) (xy 97.79 69.85)
-		)
-		(stroke
-			(width 0)
-			(type default)
-		)
-	)
 	(wire
 		(pts
@@
 	(wire
 		(pts
+			(xy 92.71 64.77) (xy 92.71 146.05)
+		)
+		(stroke
+			(width 0)
+			(type default)
+		)
+	)
+	(wire
+		(pts
 			(xy 92.71 46.99) (xy 100.33 46.99)
 		)
@@
 	(wire
 		(pts
+			(xy 97.79 44.45) (xy 97.79 69.85)
+		)
+		(stroke
+			(width 0)
+			(type default)
+		)
+	)
+	(wire
+		(pts
 			(xy 97.79 115.57) (xy 97.79 120.65)
 		)
@@
 	(wire
 		(pts
-			(xy 92.71 46.99) (xy 92.71 146.05)
-		)
-		(stroke
-			(width 0)
-			(type default)
+			(xy 92.71 46.99) (xy 92.71 57.15)
+		)
+		(stroke
+			(width 0)
+			(type default)
+		)
+	)
+	(label "GND"
+		(at 99.06 46.99 0)
+		(effects
+			(font
+				(size 1.27 1.27)
+			)
+			(justify left bottom)
+		)
+	)
+	(label "+12V"
+		(at 97.79 44.45 0)
+		(effects
+			(font
+				(size 1.27 1.27)
+			)
+			(justify left bottom)
 		)
 	)
@@
 	(symbol
 		(lib_id "Device:R_US")
-		(at 97.79 60.96 0)
+		(at 92.71 60.96 0)
 		(unit 1)
 		(body_style 1)
@@
 		(fields_autoplaced yes)
 		(property "Reference" "R1"
-			(at 100.33 59.6899 0)
+			(at 95.25 59.6899 0)
 			(show_name no)
 			(do_not_autoplace no)
@@
 		)
 		(property "Value" "73.46"
-			(at 100.33 62.2299 0)
+			(at 95.25 62.2299 0)
 			(show_name no)
 			(do_not_autoplace no)
@@
 		)
 		(property "Footprint" "Resistor_SMD:R_0805_2012Metric"
-			(at 98.806 61.214 90)
+			(at 93.726 61.214 90)
 			(hide yes)
 			(show_name no)
@@
 		)
 		(property "Datasheet" ""
-			(at 97.79 60.96 0)
+			(at 92.71 60.96 0)
 			(hide yes)
 			(show_name no)
@@
 		)
 		(property "Description" "Resistor, US symbol"
-			(at 97.79 60.96 0)
-			(hide yes)
-			(show_name no)
+			(at 92.71 60.96 0)
+			(hide yes)
+			(show_name no)
